File: PCB/hackpad.kicad_pcb (KiCad board)
At the start: 2 copper layers, 81 x 86 mm, 27 parts, among them SW1 SW_Push, SW10 SW_Push, SW11 SW_Push, SW12 SW_Push, SW2 SW_Push, SW3 SW_Push, SW4 RotaryEncoder_Switch, SW5 SW_Push, SW6 SW_Push, SW7 SW_Push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

Commit message: minor via placement change
Routing:
- net GND: track 59.4 -> 71.2 mm
Changed lines of the file:
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@@
-	)
-	(segment
-		(start 244.58 77.74263)
-		(end 233.26263 89.06)
-		(width 0.2)
-		(layer "F.Cu")
-		(net 1)
-	)
-	(segment
-		(start 233.26263 90.92737)
-		(end 231.33 92.86)
-		(width 0.2)
-		(layer "F.Cu")
-		(net 1)
 	)
 	(segment
@@
 	)
 	(segment
-		(start 231.33 92.86)
-		(end 230.306666 92.86)
+		(start 239.784 82.296)
+		(end 244.58 77.5)
 		(width 0.2)
 		(layer "F.Cu")
@@
 	)
 	(segment
-		(start 233.26263 89.06)
-		(end 233.26263 90.92737)
-		(width 0.2)
-		(layer "F.Cu")
-		(net 1)
-	)
-	(segment
-		(start 230.306666 92.86)
-		(end 230.28033 92.886336)
+		(start 231.648 82.296)
+		(end 239.784 82.296)
 		(width 0.2)
 		(layer "F.Cu")
@@
 	)
 	(via
-		(at 230.28033 92.886336)
+		(at 231.648 82.296)
 		(size 0.6)
 		(drill 0.3)
@@
 	)
 	(segment
-		(start 209.265 71.248654)
-		(end 208.591346 70.575)
+		(start 231.14 82.804)
+		(end 231.648 82.296)
 		(width 0.2)
 		(layer "B.Cu")
@@
 	)
 	(segment
-		(start 209.265 71.871006)
-		(end 209.265 71.248654)
+		(start 229.87 82.804)
+		(end 231.14 82.804)
 		(width 0.2)
 		(layer "B.Cu")
@@
 	)
 	(segment
-		(start 207.638654 70.575)
-		(end 206.965 69.901346)
+		(start 229.87 91.4)
+		(end 231.33 92.86)
 		(width 0.2)
 		(layer "B.Cu")
@@
 	)
 	(segment
-		(start 206.965 69.901346)
-		(end 206.965 68.035)
+		(start 208.115 66.885)
+		(end 205.823 66.885)
 		(width 0.2)
 		(layer "B.Cu")
@@
 	)
 	(segment
-		(start 230.28033 92.886336)
-		(end 209.265 71.871006)
+		(start 205.74 66.802)
+		(end 205.74 82.804)
 		(width 0.2)
 		(layer "B.Cu")
@@
 	)
 	(segment
-		(start 206.965 68.035)
-		(end 208.115 66.885)
+		(start 205.74 82.804)
+		(end 229.87 82.804)
 		(width 0.2)
 		(layer "B.Cu")
@@
 	)
 	(segment
-		(start 208.591346 70.575)
-		(end 207.638654 70.575)
+		(start 205.823 66.885)
+		(end 205.74 66.802)
 		(width 0.2)
 		(layer "B.Cu")
+		(net 1)
+	)
+	(segment
+		(start 229.87 82.804)
+		(end 229.87 91.4)
+		(width 0.2)
+		(layer "B.Cu")
